Commit message: add ros2_control and sim

File: ros2_src/arm_description/urdf/arm_model.xacro (robot description, xacro)
@@ -2,4 +2,5 @@
 <robot name="arm_model" xmlns:xacro="http://www.ros.org/wiki/xacro">
 <xacro:include filename="$(find arm_description)/urdf/materials.xacro" />
+<xacro:arg name="controllers_yaml" default="" />
 <!--xacro:include filename="$(find arm_description)/urdf/arm_model.trans" /-->
 <!--xacro:include filename="$(find arm_description)/urdf/arm_model.gazebo" /-->
@@ -189,4 +190,5 @@
   <child link="link_1_2_1"/>
   <axis xyz="0.0 0.0 -1.0"/>
+  <dynamics damping="1.0" friction="0.0"/>
 </joint>
 <joint name="joint_axis_2" type="continuous">
@@ -195,4 +197,5 @@
   <child link="link_2_3_1"/>
   <axis xyz="0.0 1.0 0.0"/>
+  <dynamics damping="1.0" friction="0.0"/>
 </joint>
 <joint name="joint_axis_3" type="continuous">
@@ -201,4 +204,5 @@
   <child link="link_3_4_1"/>
   <axis xyz="-0.0 -1.0 -0.0"/>
+  <dynamics damping="1.0" friction="0.0"/>
 </joint>
 <joint name="joint_finger_1" type="continuous">
@@ -207,4 +211,5 @@
   <child link="link_finger_1_1"/>
   <axis xyz="0.0 -0.866025 0.5"/>
+  <dynamics damping="1.0" friction="0.0"/>
 </joint>
 <joint name="joint_finger_2" type="continuous">
@@ -213,4 +218,5 @@
   <child link="link_finger_2_1"/>
   <axis xyz="-0.0 -0.0 -1.0"/>
+  <dynamics damping="1.0" friction="0.0"/>
 </joint>
 <joint name="joint_finger_3" type="continuous">
@@ -219,4 +225,5 @@
   <child link="link_finger_3_1"/>
   <axis xyz="0.0 0.866025 0.5"/>
+  <dynamics damping="1.0" friction="0.0"/>
 </joint>
 <joint name="joint_axis_5" type="continuous">
@@ -225,4 +232,5 @@
   <child link="link_5_endeff_1"/>
   <axis xyz="1.0 0.0 0.0"/>
+  <dynamics damping="1.0" friction="0.0"/>
 </joint>
 <joint name="joint_axis_4" type="continuous">
@@ -231,4 +239,60 @@
   <child link="link_4_5_1"/>
   <axis xyz="-0.0 1.0 0.0"/>
-</joint>
+  <dynamics damping="1.0" friction="0.0"/>
+</joint>
+<ros2_control name="ArmSystem" type="system">
+  <hardware>
+    <!-- add hardware plugin here-->
+    <!-- Gazebo Sim hardware interface -->
+    <plugin>gz_ros2_control/GazeboSimSystem</plugin>
+  </hardware>
+  <!-- List the joints ros2_control will command -->
+  <joint name="joint_axis_1">
+    <command_interface name="position"/>
+    <state_interface name="position"/>
+    <state_interface name="velocity"/>
+  </joint>
+  <joint name="joint_axis_2">
+    <command_interface name="position"/>
+    <state_interface name="position"/>
+    <state_interface name="velocity"/>
+  </joint>
+  <joint name="joint_axis_3">
+    <command_interface name="position"/>
+    <state_interface name="position"/>
+    <state_interface name="velocity"/>
+  </joint>
+  <joint name="joint_axis_4">
+    <command_interface name="position"/>
+    <state_interface name="position"/>
+    <state_interface name="velocity"/>
+  </joint>
+  <joint name="joint_axis_5">
+    <command_interface name="position"/>
+    <state_interface name="position"/>
+    <state_interface name="velocity"/>
+  </joint>
+  <joint name="joint_finger_1">
+    <command_interface name="position"/>
+    <state_interface name="position"/>
+    <state_interface name="velocity"/>
+  </joint>
+  <joint name="joint_finger_2">
+    <command_interface name="position"/>
+    <state_interface name="position"/>
+    <state_interface name="velocity"/>
+  </joint>
+  <joint name="joint_finger_3">
+    <command_interface name="position"/>
+    <state_interface name="position"/>
+    <state_interface name="velocity"/>
+  </joint>
+</ros2_control>
+<gazebo>
+  <plugin filename="gz_ros2_control-system" name="gz_ros2_control::GazeboSimROS2ControlPlugin">
+    <robot_param>robot_description</robot_param>
+    <robot_param_node>robot_state_publisher</robot_param_node>
+    <parameters>$(arg controllers_yaml)</parameters>
+  </plugin>
+</gazebo>
 </robot>
