Commit message: updated chassis description package

File: ros2_src/chassis_description/urdf/chassis_model.xacro (robot description, xacro)
@@ -1,7 +1,7 @@
 <?xml version="1.0" ?>
 <robot name="chassis_model" xmlns:xacro="http://www.ros.org/wiki/xacro">
-<xacro:include filename="$(find chassis_model_description)/urdf/materials.xacro" />
-<xacro:include filename="$(find chassis_model_description)/urdf/chassis_model.trans" />
-<xacro:include filename="$(find chassis_model_description)/urdf/chassis_model.gazebo" />
+<xacro:include filename="$(find chassis_description)/urdf/materials.xacro" />
+<xacro:include filename="$(find chassis_description)/urdf/chassis_model.trans" />
+<xacro:include filename="$(find chassis_description)/urdf/chassis_model.gazebo" />
 <link name="base_link">
   <inertial>
@@ -13,5 +13,5 @@
     <origin xyz="0 0 0" rpy="0 0 0"/>
     <geometry>
-      <mesh filename="package://chassis_model_description/meshes/base_link.stl" scale="0.001 0.001 0.001"/>
+      <mesh filename="package://chassis_description/meshes/base_link.stl" scale="0.001 0.001 0.001"/>
     </geometry>
     <material name="silver"/>
@@ -20,5 +20,5 @@
     <origin xyz="0 0 0" rpy="0 0 0"/>
     <geometry>
-      <mesh filename="package://chassis_model_description/meshes/base_link.stl" scale="0.001 0.001 0.001"/>
+      <mesh filename="package://chassis_description/meshes/base_link.stl" scale="0.001 0.001 0.001"/>
     </geometry>
   </collision>
@@ -33,5 +33,5 @@
     <origin xyz="-0.3024 0.243025 -0.0" rpy="0 0 0"/>
     <geometry>
-      <mesh filename="package://chassis_model_description/meshes/suspension_1_left_1.stl" scale="0.001 0.001 0.001"/>
+      <mesh filename="package://chassis_description/meshes/suspension_1_left_1.stl" scale="0.001 0.001 0.001"/>
     </geometry>
     <material name="silver"/>
@@ -40,5 +40,5 @@
     <origin xyz="-0.3024 0.243025 -0.0" rpy="0 0 0"/>
     <geometry>
-      <mesh filename="package://chassis_model_description/meshes/suspension_1_left_1.stl" scale="0.001 0.001 0.001"/>
+      <mesh filename="package://chassis_description/meshes/suspension_1_left_1.stl" scale="0.001 0.001 0.001"/>
     </geometry>
   </collision>
@@ -53,5 +53,5 @@
     <origin xyz="-0.3024 -0.243025 -0.0" rpy="0 0 0"/>
     <geometry>
-      <mesh filename="package://chassis_model_description/meshes/suspension_1_right_1.stl" scale="0.001 0.001 0.001"/>
+      <mesh filename="package://chassis_description/meshes/suspension_1_right_1.stl" scale="0.001 0.001 0.001"/>
     </geometry>
     <material name="silver"/>
@@ -60,5 +60,5 @@
     <origin xyz="-0.3024 -0.243025 -0.0" rpy="0 0 0"/>
     <geometry>
-      <mesh filename="package://chassis_model_description/meshes/suspension_1_right_1.stl" scale="0.001 0.001 0.001"/>
+      <mesh filename="package://chassis_description/meshes/suspension_1_right_1.stl" scale="0.001 0.001 0.001"/>
     </geometry>
   </collision>
@@ -73,5 +73,5 @@
     <origin xyz="-0.6024 0.281125 0.122" rpy="0 0 0"/>
     <geometry>
-      <mesh filename="package://chassis_model_description/meshes/suspension_2_left_1.stl" scale="0.001 0.001 0.001"/>
+      <mesh filename="package://chassis_description/meshes/suspension_2_left_1.stl" scale="0.001 0.001 0.001"/>
     </geometry>
     <material name="silver"/>
@@ -80,5 +80,5 @@
     <origin xyz="-0.6024 0.281125 0.122" rpy="0 0 0"/>
     <geometry>
-      <mesh filename="package://chassis_model_description/meshes/suspension_2_left_1.stl" scale="0.001 0.001 0.001"/>
+      <mesh filename="package://chassis_description/meshes/suspension_2_left_1.stl" scale="0.001 0.001 0.001"/>
     </geometry>
   </collision>
@@ -93,5 +93,5 @@
     <origin xyz="-0.6024 -0.281125 0.122" rpy="0 0 0"/>
     <geometry>
-      <mesh filename="package://chassis_model_description/meshes/suspension_2_right_1.stl" scale="0.001 0.001 0.001"/>
+      <mesh filename="package://chassis_description/meshes/suspension_2_right_1.stl" scale="0.001 0.001 0.001"/>
     </geometry>
     <material name="silver"/>
@@ -100,5 +100,5 @@
     <origin xyz="-0.6024 -0.281125 0.122" rpy="0 0 0"/>
     <geometry>
-      <mesh filename="package://chassis_model_description/meshes/suspension_2_right_1.stl" scale="0.001 0.001 0.001"/>
+      <mesh filename="package://chassis_description/meshes/suspension_2_right_1.stl" scale="0.001 0.001 0.001"/>
     </geometry>
   </collision>
@@ -113,5 +113,5 @@
     <origin xyz="-0.7524 0.281125 0.244" rpy="0 0 0"/>
     <geometry>
-      <mesh filename="package://chassis_model_description/meshes/wheel_3.stl" scale="0.001 0.001 0.001"/>
+      <mesh filename="package://chassis_description/meshes/wheel_3.stl" scale="0.001 0.001 0.001"/>
     </geometry>
     <material name="silver"/>
@@ -120,5 +120,5 @@
     <origin xyz="-0.7524 0.281125 0.244" rpy="0 0 0"/>
     <geometry>
-      <mesh filename="package://chassis_model_description/meshes/wheel_3.stl" scale="0.001 0.001 0.001"/>
+      <mesh filename="package://chassis_description/meshes/wheel_3.stl" scale="0.001 0.001 0.001"/>
     </geometry>
   </collision>
@@ -133,5 +133,5 @@
     <origin xyz="-0.3624 0.281125 0.244" rpy="0 0 0"/>
     <geometry>
-      <mesh filename="package://chassis_model_description/meshes/wheel_2.stl" scale="0.001 0.001 0.001"/>
+      <mesh filename="package://chassis_description/meshes/wheel_2.stl" scale="0.001 0.001 0.001"/>
     </geometry>
     <material name="silver"/>
@@ -140,5 +140,5 @@
     <origin xyz="-0.3624 0.281125 0.244" rpy="0 0 0"/>
     <geometry>
-      <mesh filename="package://chassis_model_description/meshes/wheel_2.stl" scale="0.001 0.001 0.001"/>
+      <mesh filename="package://chassis_description/meshes/wheel_2.stl" scale="0.001 0.001 0.001"/>
     </geometry>
   </collision>
@@ -153,5 +153,5 @@
     <origin xyz="0.1376 0.281125 0.244" rpy="0 0 0"/>
     <geometry>
-      <mesh filename="package://chassis_model_description/meshes/wheel_1.stl" scale="0.001 0.001 0.001"/>
+      <mesh filename="package://chassis_description/meshes/wheel_1.stl" scale="0.001 0.001 0.001"/>
     </geometry>
     <material name="silver"/>
@@ -160,5 +160,5 @@
     <origin xyz="0.1376 0.281125 0.244" rpy="0 0 0"/>
     <geometry>
-      <mesh filename="package://chassis_model_description/meshes/wheel_1.stl" scale="0.001 0.001 0.001"/>
+      <mesh filename="package://chassis_description/meshes/wheel_1.stl" scale="0.001 0.001 0.001"/>
     </geometry>
   </collision>
@@ -173,5 +173,5 @@
     <origin xyz="0.1376 -0.281125 0.244" rpy="0 0 0"/>
     <geometry>
-      <mesh filename="package://chassis_model_description/meshes/wheel_r_1.stl" scale="0.001 0.001 0.001"/>
+      <mesh filename="package://chassis_description/meshes/wheel_r_1.stl" scale="0.001 0.001 0.001"/>
     </geometry>
     <material name="silver"/>
@@ -180,5 +180,5 @@
     <origin xyz="0.1376 -0.281125 0.244" rpy="0 0 0"/>
     <geometry>
-      <mesh filename="package://chassis_model_description/meshes/wheel_r_1.stl" scale="0.001 0.001 0.001"/>
+      <mesh filename="package://chassis_description/meshes/wheel_r_1.stl" scale="0.001 0.001 0.001"/>
     </geometry>
   </collision>
@@ -193,5 +193,5 @@
     <origin xyz="-0.3624 -0.281125 0.244" rpy="0 0 0"/>
     <geometry>
-      <mesh filename="package://chassis_model_description/meshes/wheel_r_2.stl" scale="0.001 0.001 0.001"/>
+      <mesh filename="package://chassis_description/meshes/wheel_r_2.stl" scale="0.001 0.001 0.001"/>
     </geometry>
     <material name="silver"/>
@@ -200,5 +200,5 @@
     <origin xyz="-0.3624 -0.281125 0.244" rpy="0 0 0"/>
     <geometry>
-      <mesh filename="package://chassis_model_description/meshes/wheel_r_2.stl" scale="0.001 0.001 0.001"/>
+      <mesh filename="package://chassis_description/meshes/wheel_r_2.stl" scale="0.001 0.001 0.001"/>
     </geometry>
   </collision>
@@ -213,5 +213,5 @@
     <origin xyz="-0.7524 -0.281125 0.244" rpy="0 0 0"/>
     <geometry>
-      <mesh filename="package://chassis_model_description/meshes/wheel_r_3.stl" scale="0.001 0.001 0.001"/>
+      <mesh filename="package://chassis_description/meshes/wheel_r_3.stl" scale="0.001 0.001 0.001"/>
     </geometry>
     <material name="silver"/>
@@ -220,5 +220,5 @@
     <origin xyz="-0.7524 -0.281125 0.244" rpy="0 0 0"/>
     <geometry>
-      <mesh filename="package://chassis_model_description/meshes/wheel_r_3.stl" scale="0.001 0.001 0.001"/>
+      <mesh filename="package://chassis_description/meshes/wheel_r_3.stl" scale="0.001 0.001 0.001"/>
     </geometry>
   </collision>

Commit message: gazebo simulation package

File: ros2_src/chassis_description/urdf/chassis_model.xacro (robot description, xacro)
@@ -2,6 +2,6 @@
 <robot name="chassis_model" xmlns:xacro="http://www.ros.org/wiki/xacro">
 <xacro:include filename="$(find chassis_description)/urdf/materials.xacro" />
-<xacro:include filename="$(find chassis_description)/urdf/chassis_model.trans" />
-<xacro:include filename="$(find chassis_description)/urdf/chassis_model.gazebo" />
+<!--xacro:include filename="$(find chassis_description)/urdf/chassis_model.trans" /-->
+<!--xacro:include filename="$(find chassis_description)/urdf/chassis_model.gazebo" /-->
 <link name="base_link">
   <inertial>
@@ -284,3 +284,48 @@
   <axis xyz="0.0 1.0 0.0"/>
 </joint>
+<!-- ros2_control: declare command/state interfaces for wheel joints -->
+<ros2_control name="ChassisSystem" type="system">
+  <hardware>
+    <!-- Gazebo Sim hardware interface -->
+    <plugin>gz_ros2_control/GazeboSimSystem</plugin>
+  </hardware>
+  <joint name="Revolute 5">
+    <command_interface name="velocity"/>
+    <state_interface name="velocity"/>
+    <state_interface name="position"/>
+  </joint>
+  <joint name="Revolute 6">
+    <command_interface name="velocity"/>
+    <state_interface name="velocity"/>
+    <state_interface name="position"/>
+  </joint>
+  <joint name="Revolute 7">
+    <command_interface name="velocity"/>
+    <state_interface name="velocity"/>
+    <state_interface name="position"/>
+  </joint>
+  <joint name="Revolute 8">
+    <command_interface name="velocity"/>
+    <state_interface name="velocity"/>
+    <state_interface name="position"/>
+  </joint>
+  <joint name="Revolute 9">
+    <command_interface name="velocity"/>
+    <state_interface name="velocity"/>
+    <state_interface name="position"/>
+  </joint>
+  <joint name="Revolute 10">
+    <command_interface name="velocity"/>
+    <state_interface name="velocity"/>
+    <state_interface name="position"/>
+  </joint>
+</ros2_control>
+<gazebo>
+  <plugin filename="gz_ros2_control-system" name="gz_ros2_control::GazeboSimROS2ControlPlugin">
+    <robot_param>robot_description</robot_param>
+    <robot_param_node>robot_state_publisher</robot_param_node>
+    <!-- Optional: you can point to controller YAML here, or spawn controllers from launch -->
+    <!-- <parameters>$(find chassis_bringup)/config/controllers.yaml</parameters> -->
+  </plugin>
+</gazebo>
 </robot>

Commit message: Fix gazebo error

File: ros2_src/chassis_description/urdf/chassis_model.xacro (robot description, xacro)
@@ -249,5 +249,5 @@
   <axis xyz="0.0 -1.0 0.0"/>
 </joint>
-<joint name="Revolute 5" type="continuous">
+<joint name="joint_wheel_r1" type="continuous">
   <origin xyz="0.15 0.0 -0.122" rpy="0 0 0"/>
   <parent link="suspension_2_left_1"/>
@@ -255,5 +255,5 @@
   <axis xyz="0.0 -1.0 0.0"/>
 </joint>
-<joint name="Revolute 6" type="continuous">
+<joint name="joint_wheel_r2" type="continuous">
   <origin xyz="-0.24 0.0 -0.122" rpy="0 0 0"/>
   <parent link="suspension_2_left_1"/>
@@ -261,5 +261,5 @@
   <axis xyz="0.0 -1.0 0.0"/>
 </joint>
-<joint name="Revolute 7" type="continuous">
+<joint name="joint_wheel_r3" type="continuous">
   <origin xyz="-0.44 -0.0381 -0.244" rpy="0 0 0"/>
   <parent link="suspension_1_left_1"/>
@@ -267,5 +267,5 @@
   <axis xyz="0.0 -1.0 0.0"/>
 </joint>
-<joint name="Revolute 8" type="continuous">
+<joint name="joint_wheel_l1" type="continuous">
   <origin xyz="-0.44 0.0381 -0.244" rpy="0 0 0"/>
   <parent link="suspension_1_right_1"/>
@@ -273,5 +273,5 @@
   <axis xyz="0.0 1.0 0.0"/>
 </joint>
-<joint name="Revolute 9" type="continuous">
+<joint name="joint_wheel_l2" type="continuous">
   <origin xyz="-0.24 0.0 -0.122" rpy="0 0 0"/>
   <parent link="suspension_2_right_1"/>
@@ -279,5 +279,5 @@
   <axis xyz="0.0 1.0 0.0"/>
 </joint>
-<joint name="Revolute 10" type="continuous">
+<joint name="joint_wheel_l3" type="continuous">
   <origin xyz="0.15 0.0 -0.122" rpy="0 0 0"/>
   <parent link="suspension_2_right_1"/>
@@ -289,32 +289,32 @@
   <hardware>
     <!-- Gazebo Sim hardware interface -->
-    <plugin>gz_ros2_control/GazeboSimSystem</plugin>
+    <plugin>ign_ros2_control/IgnitionSystem</plugin>
   </hardware>
-  <joint name="Revolute 5">
-    <command_interface name="velocity"/>
-    <state_interface name="velocity"/>
-    <state_interface name="position"/>
-  </joint>
-  <joint name="Revolute 6">
-    <command_interface name="velocity"/>
-    <state_interface name="velocity"/>
-    <state_interface name="position"/>
-  </joint>
-  <joint name="Revolute 7">
-    <command_interface name="velocity"/>
-    <state_interface name="velocity"/>
-    <state_interface name="position"/>
-  </joint>
-  <joint name="Revolute 8">
-    <command_interface name="velocity"/>
-    <state_interface name="velocity"/>
-    <state_interface name="position"/>
-  </joint>
-  <joint name="Revolute 9">
-    <command_interface name="velocity"/>
-    <state_interface name="velocity"/>
-    <state_interface name="position"/>
-  </joint>
-  <joint name="Revolute 10">
+  <joint name="joint_wheel_r1">
+    <command_interface name="velocity"/>
+    <state_interface name="velocity"/>
+    <state_interface name="position"/>
+  </joint>
+  <joint name="joint_wheel_r2">
+    <command_interface name="velocity"/>
+    <state_interface name="velocity"/>
+    <state_interface name="position"/>
+  </joint>
+  <joint name="joint_wheel_r3">
+    <command_interface name="velocity"/>
+    <state_interface name="velocity"/>
+    <state_interface name="position"/>
+  </joint>
+  <joint name="joint_wheel_l1">
+    <command_interface name="velocity"/>
+    <state_interface name="velocity"/>
+    <state_interface name="position"/>
+  </joint>
+  <joint name="joint_wheel_l2">
+    <command_interface name="velocity"/>
+    <state_interface name="velocity"/>
+    <state_interface name="position"/>
+  </joint>
+  <joint name="joint_wheel_l3">
     <command_interface name="velocity"/>
     <state_interface name="velocity"/>
@@ -323,5 +323,5 @@
 </ros2_control>
 <gazebo>
-  <plugin filename="gz_ros2_control-system" name="gz_ros2_control::GazeboSimROS2ControlPlugin">
+  <plugin filename="ign_ros2_control-system" name="ign_ros2_control::IgnitionROS2ControlPlugin">
     <robot_param>robot_description</robot_param>
     <robot_param_node>robot_state_publisher</robot_param_node>

Commit message: change teleop to thumbstick control

File: ros2_src/chassis_description/urdf/chassis_model.xacro (robot description, xacro)
@@ -225,5 +225,5 @@
   </collision>
 </link>
-<joint name="Revolute 1" type="continuous">
+<joint name="Revolute 1" type="fixed">
   <origin xyz="0.3024 -0.243025 0.0" rpy="0 0 0"/>
   <parent link="base_link"/>
@@ -231,5 +231,5 @@
   <axis xyz="0.0 1.0 0.0"/>
 </joint>
-<joint name="Revolute 2" type="continuous">
+<joint name="Revolute 2" type="fixed">
   <origin xyz="0.3024 0.243025 0.0" rpy="0 0 0"/>
   <parent link="base_link"/>
@@ -237,5 +237,5 @@
   <axis xyz="0.0 1.0 0.0"/>
 </joint>
-<joint name="Revolute 3" type="continuous">
+<joint name="Revolute 3" type="fixed">
   <origin xyz="0.3 -0.0381 -0.122" rpy="0 0 0"/>
   <parent link="suspension_1_left_1"/>
@@ -243,5 +243,5 @@
   <axis xyz="0.0 1.0 0.0"/>
 </joint>
-<joint name="Revolute 4" type="continuous">
+<joint name="Revolute 4" type="fixed">
   <origin xyz="0.3 0.0381 -0.122" rpy="0 0 0"/>
   <parent link="suspension_1_right_1"/>
@@ -253,5 +253,5 @@
   <parent link="suspension_2_left_1"/>
   <child link="wheel_3"/>
-  <axis xyz="0.0 -1.0 0.0"/>
+  <axis xyz="0.0 1.0 0.0"/>
 </joint>
 <joint name="joint_wheel_r2" type="continuous">
@@ -259,5 +259,5 @@
   <parent link="suspension_2_left_1"/>
   <child link="wheel_2"/>
-  <axis xyz="0.0 -1.0 0.0"/>
+  <axis xyz="0.0 1.0 0.0"/>
 </joint>
 <joint name="joint_wheel_r3" type="continuous">
@@ -265,5 +265,5 @@
   <parent link="suspension_1_left_1"/>
   <child link="wheel_1"/>
-  <axis xyz="0.0 -1.0 0.0"/>
+  <axis xyz="0.0 1.0 0.0"/>
 </joint>
 <joint name="joint_wheel_l1" type="continuous">

Commit message: fix chassis x axis by adding new base link and rotating

File: ros2_src/chassis_description/urdf/chassis_model.xacro (robot description, xacro)
@@ -5,4 +5,12 @@
 <!--xacro:include filename="$(find chassis_description)/urdf/chassis_model.trans" /-->
 <!--xacro:include filename="$(find chassis_description)/urdf/chassis_model.gazebo" /-->
+<!-- Root frame aligned with ROS conventions (+X forward, +Y left, +Z up) -->
+<link name="base_footprint"/>
+<!-- CAD export had base_link facing opposite X; rotate by pi around Z -->
+<joint name="base_footprint_to_base_link" type="fixed">
+  <origin xyz="0 0 0" rpy="0 0 3.141592653589793"/>
+  <parent link="base_footprint"/>
+  <child link="base_link"/>
+</joint>
 <link name="base_link">
   <inertial>
@@ -323,11 +331,11 @@
 </ros2_control>
 <xacro:include filename="$(find chassis_description)/urdf/chassis_sensors.gazebo.xacro"/>
-<xacro:add_imu_sensor parent="base_link" imu_link="imu_link"
+<xacro:add_imu_sensor parent="base_footprint" imu_link="imu_link"
                           xyz="0.0 0.0 0.15" rpy="0 0 0"
                           topic="/imu" rate="200"/>
-    <xacro:add_gps_sensor parent="base_link" gps_link="gps_link"
+    <xacro:add_gps_sensor parent="base_footprint" gps_link="gps_link"
                           xyz="0.0 0.0 0.30" rpy="0 0 0"
                           topic="/navsat" rate="10"/>
-    <xacro:add_depth_camera parent="base_link"
+    <xacro:add_depth_camera parent="base_footprint"
                             cam_link="camera_link"
                             optical_link="camera_optical_frame"

Commit message: fix wheel joint signs so cmd vel postive is forward

File: ros2_src/chassis_description/urdf/chassis_model.xacro (robot description, xacro)
@@ -259,37 +259,37 @@
 <joint name="joint_wheel_r1" type="continuous">
   <origin xyz="0.15 0.0 -0.122" rpy="0 0 0"/>
-  <parent link="suspension_2_left_1"/>
-  <child link="wheel_3"/>
-  <axis xyz="0.0 1.0 0.0"/>
+  <parent link="suspension_2_right_1"/>
+  <child link="wheel_r_1"/>
+  <axis xyz="0.0 -1.0 0.0"/>
 </joint>
 <joint name="joint_wheel_r2" type="continuous">
+  <origin xyz="-0.24 0.0 -0.122" rpy="0 0 0"/>
+  <parent link="suspension_2_right_1"/>
+  <child link="wheel_r_2"/>
+  <axis xyz="0.0 -1.0 0.0"/>
+</joint>
+<joint name="joint_wheel_r3" type="continuous">
+  <origin xyz="-0.44 0 -0.244" rpy="0 0 0"/>
+  <parent link="suspension_1_right_1"/>
+  <child link="wheel_r_3"/>
+  <axis xyz="0.0 -1.0 0.0"/>
+</joint>
+<joint name="joint_wheel_l1" type="continuous">
+  <origin xyz="-0.44 0 -0.244" rpy="0 0 0"/>
+  <parent link="suspension_1_left_1"/>
+  <child link="wheel_1"/>
+  <axis xyz="0.0 -1.0 0.0"/>
+</joint>
+<joint name="joint_wheel_l2" type="continuous">
   <origin xyz="-0.24 0.0 -0.122" rpy="0 0 0"/>
   <parent link="suspension_2_left_1"/>
   <child link="wheel_2"/>
-  <axis xyz="0.0 1.0 0.0"/>
-</joint>
-<joint name="joint_wheel_r3" type="continuous">
-  <origin xyz="-0.44 -0.0381 -0.244" rpy="0 0 0"/>
-  <parent link="suspension_1_left_1"/>
-  <child link="wheel_1"/>
-  <axis xyz="0.0 1.0 0.0"/>
-</joint>
-<joint name="joint_wheel_l1" type="continuous">
-  <origin xyz="-0.44 0.0381 -0.244" rpy="0 0 0"/>
-  <parent link="suspension_1_right_1"/>
-  <child link="wheel_r_1"/>
-  <axis xyz="0.0 1.0 0.0"/>
-</joint>
-<joint name="joint_wheel_l2" type="continuous">
-  <origin xyz="-0.24 0.0 -0.122" rpy="0 0 0"/>
-  <parent link="suspension_2_right_1"/>
-  <child link="wheel_r_2"/>
-  <axis xyz="0.0 1.0 0.0"/>
+  <axis xyz="0.0 -1.0 0.0"/>
 </joint>
 <joint name="joint_wheel_l3" type="continuous">
   <origin xyz="0.15 0.0 -0.122" rpy="0 0 0"/>
-  <parent link="suspension_2_right_1"/>
-  <child link="wheel_r_3"/>
-  <axis xyz="0.0 1.0 0.0"/>
+  <parent link="suspension_2_left_1"/>
+  <child link="wheel_3"/>
+  <axis xyz="0.0 -1.0 0.0"/>
 </joint>
 <!-- ros2_control: declare command/state interfaces for wheel joints -->
